Commit message: first commit

File: src/rocker_description/urdf/rocker.urdf.xacro (robot description, xacro)
@@ -1,889 +1,397 @@
 <?xml version="1.0" encoding="utf-8"?>
-<!-- This URDF was automatically created by SolidWorks to URDF Exporter! Originally created by Stephen Brawner (brawner@gmail.com)
-     Commit Version: 1.6.0-4-g7f85cfe  Build Version: 1.6.7995.38578
-     For more information, please see http://wiki.ros.org/sw_urdf_exporter -->
 <robot name="rocker" xmlns:xacro="http://ros.org/wiki/xacro">
-  <!-- Start GZ or Ignition depending on ROS 2 Version -->
   <xacro:arg name="is_ignition" default="true"/>
-  <!-- Include Gazebo Parameters -->
   <xacro:include filename="$(find rocker_description)/urdf/rocker_gazebo.xacro" />
-  <!-- Include control -->
   <xacro:include filename="$(find rocker_description)/urdf/rocker_ros2_control.xacro"/>
-  <link
-    name="base_link">
-    <inertial>
-      <origin
-        xyz="0.0036425 -1.0237E-05 0.029007"
-        rpy="0 0 0" />
-      <mass
-        value="3.2505" />
-      <inertia
-        ixx="0.012194"
-        ixy="-1.2887E-11"
-        ixz="-1.2673E-05"
-        iyy="0.0094514"
-        iyz="2.0372E-12"
-        izz="0.019133" />
-    </inertial>
-    <visual>
-      <origin
-        xyz="0 0 0"
-        rpy="0 0 0" />
-      <geometry>
-        <mesh
-          filename="package://rocker_description/meshes/base_link.STL" />
-      </geometry>
-      <material
-        name="">
-        <color
-          rgba="1 0 0 1" />
-      </material>
-    </visual>
-    <collision>
-      <origin
-        xyz="0 0 0"
-        rpy="0 0 0" />
-      <geometry>
-        <mesh
-          filename="package://rocker_description/meshes/base_link.STL" />
-      </geometry>
-    </collision>
-  </link>
-  <link
-    name="rocker_left">
-    <inertial>
-      <origin
-        xyz="-0.00596279660858899 0.019311656764223 0.00821775119149987"
-        rpy="0 0 0" />
-      <mass
-        value="0.548279465838668" />
-      <inertia
-        ixx="0.000160712183052689"
-        ixy="-1.18295174930768E-05"
-        ixz="4.65341223670499E-08"
-        iyy="0.00145712336712729"
-        iyz="2.38546500296045E-06"
-        izz="0.00150112676272773" />
-    </inertial>
-    <visual>
-      <origin
-        xyz="0 0 0"
-        rpy="0 0 0" />
-      <geometry>
-        <mesh
-          filename="package://rocker_description/meshes/rocker_left.STL" />
-      </geometry>
-      <material
-        name="">
-        <color
-          rgba="0.752941176470588 0.752941176470588 0.752941176470588 1" />
-      </material>
-    </visual>
-    <collision>
-      <origin
-        xyz="0 0 0"
-        rpy="0 0 0" />
-      <geometry>
-        <mesh
-          filename="package://rocker_description/meshes/rocker_left.STL" />
-      </geometry>
-    </collision>
-  </link>
-  <joint
-    name="rocker_left_joint"
-    type="revolute">
-    <origin
-      xyz="-0.00300007366280326 0.139989762643875 0.00599815142431871"
-      rpy="-1.5707963267949 0 0" />
-    <parent
-      link="base_link" />
-    <child
-      link="rocker_left" />
-    <axis
-      xyz="0 0 -1" />
-    <limit
-      lower="-0.785"
-      upper="0.785"
-      effort="10"
-      velocity="20" />
-  </joint>
-  <link
-    name="steer_fl">
-    <inertial>
-      <origin
-        xyz="0.000519302762488599 0.00116147480983056 -0.0722490116852784"
-        rpy="0 0 0" />
-      <mass
-        value="0.0538768863875911" />
-      <inertia
-        ixx="1.72835692168003E-05"
-        ixy="1.86520451951073E-10"
-        ixz="1.22945601642171E-09"
-        iyy="1.26504996734862E-05"
-        iyz="1.03486603556425E-12"
-        izz="1.01151748087639E-05" />
-    </inertial>
-    <visual>
-      <origin
-        xyz="0 0 0"
-        rpy="0 0 0" />
-      <geometry>
-        <mesh
-          filename="package://rocker_description/meshes/steer_fl.STL" />
-      </geometry>
-      <material
-        name="">
-        <color
-          rgba="0.752941176470588 0.752941176470588 0.752941176470588 1" />
-      </material>
-    </visual>
-    <collision>
-      <origin
-        xyz="0 0 0"
-        rpy="0 0 0" />
-      <geometry>
-        <mesh
-          filename="package://rocker_description/meshes/steer_fl.STL" />
-      </geometry>
-    </collision>
-  </link>
-  <joint
-    name="steer_fl_joint"
-    type="revolute">
-    <origin
-      xyz="0.109493624388031 0.03794110103799 0.0465656792826112"
-      rpy="1.5707963267949 0 0" />
-    <parent
-      link="rocker_left" />
-    <child
-      link="steer_fl" />
-    <axis
-      xyz="0 0 -1" />
-    <limit
-      lower="-3.14"
-      upper="3.14"
-      effort="10"
-      velocity="20" />
-  </joint>
-  <link
-    name="fl_wheel">
-    <inertial>
-      <origin
-        xyz="0.002099 -0.0019395 -0.028409"
-        rpy="0 0 0" />
-      <mass
-        value="0.13017" />
-      <inertia
-        ixx="0.00012478"
-        ixy="-7.5675E-12"
-        ixz="-1.0928E-11"
-        iyy="0.00012478"
-        iyz="-2.364E-12"
-        izz="0.00023467" />
-    </inertial>
-    <visual>
-      <origin
-        xyz="0 0 0"
-        rpy="0 0 0" />
-      <geometry>
-        <mesh
-          filename="package://rocker_description/meshes/fl_wheel.STL" />
-      </geometry>
-      <material
-        name="">
-        <color
-          rgba="0 0 0 1" />
-      </material>
-    </visual>
-    <collision>
-      <origin
-        xyz="0 0 0"
-        rpy="0 0 0" />
-      <geometry>
-        <mesh
-          filename="package://rocker_description/meshes/fl_wheel.STL" />
-      </geometry>
-    </collision>
-  </link>
-  <joint
-    name="fl_wheel_joint"
-    type="continuous">
-    <origin
-      xyz="-0.0015781170593388 0.0908967088232542 -0.0809547532967621"
-      rpy="-1.5707963267949 0 0" />
-    <parent
-      link="steer_fl" />
-    <child
-      link="fl_wheel" />
-    <axis
-      xyz="0 0 -1" />
-    <limit
-      lower="-10"
-      upper="10"
-      effort="10"
-      velocity="100" />
-  </joint>
-  <link
-    name="steer_rl">
-    <inertial>
-      <origin
-        xyz="0.000484941628677482 0.00116147483099063 -0.0761644404434853"
-        rpy="0 0 0" />
-      <mass
-        value="0.053876886763219" />
-      <inertia
-        ixx="1.72835692136404E-05"
-        ixy="1.8652062791263E-10"
-        ixz="1.22944997559593E-09"
-        iyy="1.26504996782381E-05"
-        iyz="1.04212079064367E-12"
-        izz="1.01151748208476E-05" />
-    </inertial>
-    <visual>
-      <origin
-        xyz="0 0 0"
-        rpy="0 0 0" />
-      <geometry>
-        <mesh
-          filename="package://rocker_description/meshes/steer_rl.STL" />
-      </geometry>
-      <material
-        name="">
-        <color
-          rgba="0.752941176470588 0.752941176470588 0.752941176470588 1" />
-      </material>
-    </visual>
-    <collision>
-      <origin
-        xyz="0 0 0"
-        rpy="0 0 0" />
-      <geometry>
-        <mesh
-          filename="package://rocker_description/meshes/steer_rl.STL" />
-      </geometry>
-    </collision>
-  </link>
-  <joint
-    name="steer_rl_joint"
-    type="revolute">
-    <origin
-      xyz="-0.110472012747799 0.0340528521482858 0.0465656792826093"
-      rpy="1.5707963267949 0 0" />
-    <parent
-      link="rocker_left" />
-    <child
-      link="steer_rl" />
-    <axis
-      xyz="0 0 -1" />
-    <limit
-      lower="-3.14"
-      upper="3.14"
-      effort="10"
-      velocity="20" />
-  </joint>
-  <link
-    name="rl_wheel">
-    <inertial>
-      <origin
-        xyz="0.0020646 0.001976 -0.028409"
-        rpy="0 0 0" />
-      <mass
-        value="0.13017" />
-      <inertia
-        ixx="0.00012478"
-        ixy="3.8397E-11"
-        ixz="1.7184E-12"
-        iyy="0.00012478"
-        iyz="1.1048E-11"
-        izz="0.00023467" />
-    </inertial>
-    <visual>
-      <origin
-        xyz="0 0 0"
-        rpy="0 0 0" />
-      <geometry>
-        <mesh
-          filename="package://rocker_description/meshes/rl_wheel.STL" />
-      </geometry>
-      <material
-        name="">
-        <color
-          rgba="0 0 0 1" />
-      </material>
-    </visual>
-    <collision>
-      <origin
-        xyz="0 0 0"
-        rpy="0 0 0" />
-      <geometry>
-        <mesh
-          filename="package://rocker_description/meshes/rl_wheel.STL" />
-      </geometry>
-    </collision>
-  </link>
-  <joint
-    name="rl_wheel_joint"
-    type="continuous">
-    <origin
-      xyz="-0.00157811705934295 0.0908967088232554 -0.0809547532967675"
-      rpy="-1.5707963267949 0 0" />
-    <parent
-      link="steer_rl" />
-    <child
-      link="rl_wheel" />
-    <axis
-      xyz="0 0 -1" />
-    <limit
-      lower="-10"
-      upper="10"
-      effort="10"
-      velocity="100" />
-  </joint>
-  <link
-    name="rocker_right">
-    <inertial>
-      <origin
-        xyz="-0.00596288564139164 -0.0193116567738485 0.00817977279760604"
-        rpy="0 0 0" />
-      <mass
-        value="0.54827946587469" />
-      <inertia
-        ixx="0.000160712214952262"
-        ixy="1.17004377021412E-05"
-        ixz="-4.595305488417E-08"
-        iyy="0.00145712333524181"
-        iyz="-2.31782014461646E-06"
-        izz="0.00150112676273801" />
-    </inertial>
-    <visual>
-      <origin
-        xyz="0 0 0"
-        rpy="0 0 0" />
-      <geometry>
-        <mesh
-          filename="package://rocker_description/meshes/rocker_right.STL" />
-      </geometry>
-      <material
-        name="">
-        <color
-          rgba="0.752941176470588 0.752941176470588 0.752941176470588 1" />
-      </material>
-    </visual>
-    <collision>
-      <origin
-        xyz="0 0 0"
-        rpy="0 0 0" />
-      <geometry>
-        <mesh
-          filename="package://rocker_description/meshes/rocker_right.STL" />
-      </geometry>
-    </collision>
-  </link>
-  <joint
-    name="rocker_right_joint"
-    type="revolute">
-    <origin
-      xyz="-0.00300007366280228 -0.140010237356125 0.00599815142431871"
-      rpy="1.5707963267949 0 0" />
-    <parent
-      link="base_link" />
-    <child
-      link="rocker_right" />
-    <axis
-      xyz="0 0 -1" />
-    <limit
-      lower="-0.785"
-      upper="0.785"
-      effort="10"
-      velocity="20" />
-  </joint>
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
File: src/rocker_description/urdf/rocker_gazebo.xacro (robot description, xacro)
@@ -1,5 +1,4 @@
 <?xml version="1.0"?>
 <robot name="rocker" xmlns:xacro="http://ros.org/wiki/xacro">
-  <!-- Wheels -->
   <gazebo reference="fl_wheel">
     <mu1>1.0</mu1>
@@ -63,27 +62,40 @@
   </gazebo>
   <gazebo>
-    <!-- ROS 2 Control Plugin -->
-    <plugin filename="ign_ros2_control-system" name="ign_ros2_control::IgnitionROS2ControlPlugin">
-      <parameters>$(find rocker_controller)/config/rocker_controllers.yaml</parameters>
-    </plugin>
-    <!-- IMU Sensor System -->
-    <plugin filename="ignition-gazebo-imu-system" name="ignition::gazebo::systems::Imu"/>
-    <!-- Sensor Management System -->
-    <plugin filename="ignition-gazebo-sensors-system" name="ignition::gazebo::systems::Sensors"/>
+    <xacro:if value="$(arg is_ignition)">
+      <plugin name="ign_ros2_control::IgnitionROS2ControlPlugin" filename="ign_ros2_control-system">
+        <parameters>$(find rocker_controller)/config/rocker_controllers.yaml</parameters>
+      </plugin>
+      <plugin name="ignition::gazebo::systems::Imu" filename="ignition-gazebo-imu-system" />
+      <plugin name="ignition::gazebo::systems::Sensors" filename="ignition-gazebo-sensors-system">
+        <render_engine>ogre2</render_engine>
+      </plugin>
+    </xacro:if>
+    <xacro:unless value="$(arg is_ignition)">
+      <plugin name="gz_ros2_control::GazeboSimROS2ControlPlugin" filename="gz_ros2_control-system">
+        <parameters>$(find rocker_controller)/config/rocker_controllers.yaml</parameters>
+      </plugin>
+      <plugin name="gz::sim::systems::Imu" filename="gz-sim-imu-system" />
+      <plugin name="gz::sim::systems::Sensors" filename="gz-sim-sensors-system">
+        <render_engine>ogre2</render_engine>
+      </plugin>
+    </xacro:unless>
   </gazebo>
-  <!-- Detachable Joint Plugin to Simulate Multi-Parent (e.g., 4-bar style) -->
   <gazebo>
-    <plugin filename="libgz-sim-detachable-joint-system.so" name="gz::sim::systems::DetachableJoint">
-      <parent_link>rocker_left</parent_link>
-      <child_model>bot</child_model>
-      <child_link>turnbuckle_left</child_link>
-      <attach_topic>attach_diff_to_left</attach_topic>
-    </plugin>
-    <plugin filename="libgz-sim-detachable-joint-system.so" name="gz::sim::systems::DetachableJoint">
-      <parent_link>rocker_right</parent_link>
-      <child_model>bot</child_model>
-      <child_link>turnbuckle_right</child_link>
-      <attach_topic>attach_diff_to_right</attach_topic>
-    </plugin>
-  </gazebo>
+  <plugin filename="libgz-sim-detachable-joint-system.so" name="gz::sim::systems::DetachableJoint">
+    <parent_link>rocker_left</parent_link>
+    <child_model>bot</child_model>
+    <child_link>turnbuckle_left</child_link>
+    <detach_topic>detach_diff_from_left</detach_topic>
+    <attach_topic>attach_diff_to_left</attach_topic>
+    <output_topic>left_detach_status</output_topic>
+  </plugin>
+  <plugin filename="libgz-sim-detachable-joint-system.so" name="gz::sim::systems::DetachableJoint">
+    <parent_link>rocker_right</parent_link>
+    <child_model>bot</child_model>
+    <child_link>turnbuckle_right</child_link>
+    <detach_topic>detach_diff_from_right</detach_topic>
+    <attach_topic>attach_diff_to_right</attach_topic>
+    <output_topic>right_detach_status</output_topic>
+  </plugin>
+</gazebo>
 </robot>

File: src/rocker_description/urdf/rocker_ros2_control.xacro (robot description, xacro)
@@ -1,5 +1,4 @@
 <?xml version="1.0"?>
 <robot name="rocker" xmlns:xacro="http://ros.org/wiki/xacro">
-  <!-- Declare missing arguments -->
   <xacro:arg name="is_sim" default="true"/>
   <xacro:arg name="is_ignition" default="true"/>
@@ -10,5 +9,4 @@
       </hardware>
     </xacro:if>
-    <!-- DRIVE WHEEL JOINTS (VELOCITY CONTROL) -->
     <joint name="fr_wheel_joint">
       <command_interface name="velocity">
@@ -43,5 +41,4 @@
       <state_interface name="velocity"/>
     </joint>
-    <!-- STEERING JOINTS (POSITION CONTROL) -->
     <joint name="steer_fl_joint">
       <command_interface name="position"/>
@@ -64,4 +61,14 @@
       <state_interface name="velocity"/>
     </joint>
+    <joint name="rocker_left_joint">
+      <command_interface name="position"/>
+      <state_interface name="position"/>
+      <state_interface name="velocity"/>
+    </joint>
+    <joint name="rocker_right_joint">
+      <command_interface name="position"/>
+      <state_interface name="position"/>
+      <state_interface name="velocity"/>
+    </joint>
   </ros2_control>
 </robot>
